File: URC OH Front Panel/URC OH Front Panel.kicad_pcb (KiCad board)
At the start: 2 copper layers, 88 x 38 mm, 2 parts

Commit message: locked switch location
Other:
- board text added: "Suggested location of switch hole"
Changed lines of the file:
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@@
   (gr_circle locked (center 99.45 83.775) (end 102 83.775)
     (stroke (width 0.1) (type default)) (fill none) (layer "Edge.Cuts"))
-  (gr_rect (start 65.125 69.85) (end 71.425 72.05)
+  (gr_rect locked (start 65.125 69.85) (end 71.425 72.05)
     (stroke (width 0.15) (type default)) (fill none) (layer "Edge.Cuts"))
   (gr_circle locked (center 66.45 83.775) (end 69 83.775)
@@
     (effects (font (size 1 1) (thickness 0.15)) (justify left bottom))
   )
+  (gr_text "Suggested location of\nswitch hole" (at 52.1 72.3) (layer "Cmts.User")
+    (effects (font (size 1 1) (thickness 0.15)) (justify bottom))
+  )
   (gr_text "Retain for JLC order number\ncustom location\n" (at 91.4 55.9) (layer "Cmts.User")
